Commit message: add lidar

File: description/colors.xacro (robot description, xacro)
@@ -13,3 +13,6 @@
         <color rgba="0 0 0 1" />
     </material>
+    <material name="red">
+        <color rgba="1 0 0 1" />
+    </material>
 </robot>

Commit message: add gazebo clolors

File: description/colors.xacro (robot description, xacro)
@@ -16,3 +16,17 @@
         <color rgba="1 0 0 1" />
     </material>
+    <gazebo reference="chassis">
+        <material>Gazebo/White</material>
+    </gazebo>
+    <gazebo reference="left_wheel">
+        <material>Gazebo/Blue</material>
+    </gazebo>
+    <gazebo reference="right_wheel">
+        <material>Gazebo/Blue</material>
+    </gazebo>
+    <gazebo reference="caster_wheel">
+        <material>Gazebo/Black</material>
+        <mu1 value="0.001" />
+        <mu2 value="0.001" />
+    </gazebo>
 </robot>
