Commit message: add ros2_control

File: description/camera.xacro (robot description, xacro)
@@ -4,5 +4,5 @@
         <parent link="chassis" />
         <child link="camera_link" />
-        <origin xyz="0.305 0 0.08" rpy="0 0 0" />
+        <origin xyz="0.276 0 0.181" rpy="0 0.18 0" />
     </joint>
     <link name="camera_link">
@@ -11,5 +11,12 @@
                 <box size="0.010 0.03 0.03" />
             </geometry>
-            <material name="red" />
+            <material name="black" />
+        </visual>
+        <visual>
+            <origin xyz="0 0 -0.05" />
+            <geometry>
+                <cylinder radius="0.002" length="0.1" />
+            </geometry>
+            <material name="black" />
         </visual>
     </link>
@@ -17,9 +24,9 @@
         <parent link="camera_link" />
         <child link="camera_link_optical" />
-        <origin xyz="0 0 00" rpy="${-pi/2} 0 ${-pi/2}" />
+        <origin xyz="0 0 0" rpy="${-pi/2} 0 ${-pi/2}" />
     </joint>
-    <link name="camera_link_optical" />
+    <link name="camera_link_optical"></link>
     <gazebo reference="camera_link">
-        <material>Gazebo/Red</material>
+        <material>Gazebo/Black</material>
         <sensor name="camera" type="camera">
             <pose> 0 0 0 0 0 0 </pose>
@@ -32,9 +39,9 @@
                     <width>640</width>
                     <height>480</height>
-                    <clip>
-                        <near>0.05</near>
-                        <far>8.0</far>
-                    </clip>
                 </image>
+                <clip>
+                    <near>0.05</near>
+                    <far>8.0</far>
+                </clip>
             </camera>
             <plugin name="camera_controller" filename="libgazebo_ros_camera.so">

File: description/colors.xacro (robot description, xacro)
@@ -17,5 +17,5 @@
     </material>
     <gazebo reference="chassis">
-        <material>Gazebo/White</material>
+        <material>Gazebo/Orange</material>
     </gazebo>
     <gazebo reference="left_wheel">

File: description/lidar.xacro (robot description, xacro)
@@ -4,5 +4,5 @@
         <parent link="chassis" />
         <child link="laser_frame" />
-        <origin xyz="0.1 0 0.175" rpy="0 0 0" />
+        <origin xyz="0.122 0 0.212" rpy="0 0 0" />
     </joint>
     <link name="laser_frame">
@@ -11,5 +11,12 @@
                 <cylinder radius="0.05" length="0.04" />
             </geometry>
-            <material name="red" />
+            <material name="black" />
+        </visual>
+        <visual>
+            <origin xyz="0 0 -0.05" />
+            <geometry>
+                <cylinder radius="0.01" length="0.1" />
+            </geometry>
+            <material name="black" />
         </visual>
         <collision>
@@ -23,5 +30,5 @@
     </link>
     <gazebo reference="laser_frame">
-        <material>Gazebo/Red</material>
+        <material>Gazebo/Black</material>
         <sensor name="laser" type="ray">
             <pose> 0 0 0 0 0 0 </pose>

File: description/robot.urdf.xacro (robot description, xacro)
@@ -1,8 +1,15 @@
 <?xml version="1.0"?>
 <robot xmlns:xacro="http://www.ros.org/wiki/xacro"  name="robot">
+    <xacro:arg name="use_ros2_control" default="true" />
     <xacro:include filename="robot_core.xacro" />
-    <xacro:include filename="gazebo_control.xacro" />
+    <xacro:if value="$(arg use_ros2_control)">
+        <xacro:include filename="ros2_control.xacro" />
+    </xacro:if>
+    <xacro:unless value="$(arg use_ros2_control)">
+        <xacro:include filename="gazebo_control.xacro" />
+    </xacro:unless>
     <xacro:include filename="lidar.xacro" />
-    <!-- <xacro:include filename="camera.xacro" /> -->
-    <xacro:include filename="depth_camera.xacro" />
+    <xacro:include filename="camera.xacro" />
+    <xacro:include filename="face.xacro" />
+    <!-- <xacro:include filename="depth_camera.xacro" /> -->
 </robot>

File: description/robot_core.xacro (robot description, xacro)
@@ -3,36 +3,60 @@
     <xacro:include filename="colors.xacro" />
     <xacro:include filename="inertial_macros.xacro" />
-    <!-- Base Link -->
+    <xacro:property name="chassis_length" value="0.335" />
+    <xacro:property name="chassis_width" value="0.265" />
+    <xacro:property name="chassis_height" value="0.138" />
+    <xacro:property name="chassis_mass" value="1.0" />
+    <xacro:property name="wheel_radius" value="0.033" />
+    <xacro:property name="wheel_thickness" value="0.026" />
+    <xacro:property name="wheel_mass" value="0.05" />
+    <xacro:property name="wheel_offset_x" value="0.226" />
+    <xacro:property name="wheel_offset_y" value="0.1485" />
+    <xacro:property name="wheel_offset_z" value="0.01" />
+    <xacro:property name="caster_wheel_radius" value="0.01" />
+    <xacro:property name="caster_wheel_mass" value="0.01" />
+    <xacro:property name="caster_wheel_offset_x" value="0.075" />
+    <xacro:property name="caster_wheel_offset_z"
+        value="${wheel_offset_z - wheel_radius + caster_wheel_radius}" />
+    <!-- BASE LINK -->
     <link name="base_link">
     </link>
-    <!-- Chassis Link -->
+    <!-- BASE_FOOTPRINT LINK -->
+    <joint name="base_footprint_joint" type="fixed">
+        <parent link="base_link" />
+        <child link="base_footprint" />
+        <origin xyz="0 0 0" rpy="0 0 0" />
+    </joint>
+    <link name="base_footprint">
+    </link>
+    <!-- CHASSIS LINK -->
     <joint name="chassis_joint" type="fixed">
         <parent link="base_link" />
         <child link="chassis" />
-        <origin xyz="-0.1 0 0" />
+        <origin xyz="${-wheel_offset_x} 0 ${-wheel_offset_z}" />
     </joint>
     <link name="chassis">
         <visual>
-            <origin xyz="0.15 0 0.075" />
+            <origin xyz="${chassis_length/2} 0 ${chassis_height/2}" />
             <geometry>
-                <box size="0.3 0.3 0.15" />
+                <box size="${chassis_length} ${chassis_width} ${chassis_height}" />
             </geometry>
-            <material name="white" />
+            <material name="orange" />
         </visual>
         <collision>
-            <origin xyz="0.15 0 0.075" />
+            <origin xyz="${chassis_length/2} 0 ${chassis_height/2}" />
             <geometry>
-                <box size="0.3 0.3 0.15" />
+                <box size="${chassis_length} ${chassis_width} ${chassis_height}" />
             </geometry>
         </collision>
-        <xacro:inertial_box mass="0.5" x="0.3" y="0.3" z="0.15">
-            <origin xyz="0.15 0 0.075" rpy="0 0 0" />
+        <xacro:inertial_box mass="0.5" x="${chassis_length}" y="${chassis_width}"
+            z="${chassis_height}">
+            <origin xyz="${chassis_length/2} 0 ${chassis_height/2}" rpy="0 0 0" />
         </xacro:inertial_box>
     </link>
-    <!-- Left Wheel Link -->
+    <!-- LEFT WHEEL LINK -->
     <joint name="left_wheel_joint" type="continuous">
         <parent link="base_link" />
         <child link="left_wheel" />
-        <origin xyz="0 0.175 0" rpy="-${pi/2} 0 0" />
+        <origin xyz="0 ${wheel_offset_y} 0" rpy="-${pi/2} 0 0" />
         <axis xyz="0 0 1" />
     </joint>
@@ -40,5 +64,5 @@
         <visual>
             <geometry>
-                <cylinder radius="0.05" length="0.04" />
+                <cylinder radius="${wheel_radius}" length="${wheel_thickness}" />
             </geometry>
             <material name="blue" />
@@ -46,16 +70,17 @@
         <collision>
             <geometry>
-                <cylinder radius="0.05" length="0.04" />
+                <sphere radius="${wheel_radius}" />
             </geometry>
         </collision>
-        <xacro:inertial_cylinder mass="0.1" length="0.04" radius="0.05">
+        <xacro:inertial_cylinder mass="${wheel_mass}" length="${wheel_thickness}"
+            radius="${wheel_radius}">
             <origin xyz="0 0 0" rpy="0 0 0" />
         </xacro:inertial_cylinder>
     </link>
-    <!-- Right Wheel Link -->
+    <!-- RIGHT WHEEL LINK -->
     <joint name="right_wheel_joint" type="continuous">
         <parent link="base_link" />
         <child link="right_wheel" />
-        <origin xyz="0 -0.175 0" rpy="${pi/2} 0 0" />
+        <origin xyz="0 ${-wheel_offset_y} 0" rpy="${pi/2} 0 0" />
         <axis xyz="0 0 -1" />
     </joint>
@@ -63,5 +88,5 @@
         <visual>
             <geometry>
-                <cylinder radius="0.05" length="0.04" />
+                <cylinder radius="${wheel_radius}" length="${wheel_thickness}" />
             </geometry>
             <material name="blue" />
@@ -69,30 +94,31 @@
         <collision>
             <geometry>
-                <cylinder radius="0.05" length="0.04" />
+                <sphere radius="${wheel_radius}" />
             </geometry>
         </collision>
-        <xacro:inertial_cylinder mass="0.1" length="0.04" radius="0.05">
+        <xacro:inertial_cylinder mass="${wheel_mass}" length="${wheel_thickness}"
+            radius="${wheel_radius}">
             <origin xyz="0 0 0" rpy="0 0 0" />
         </xacro:inertial_cylinder>
     </link>
-    <!-- Caster Wheel -->
+    <!-- CASTER WHEEL LINK -->
     <joint name="caster_wheel_joint" type="fixed">
         <parent link="chassis" />
         <child link="caster_wheel" />
-        <origin xyz="0.24 0 0" />
+        <origin xyz="${caster_wheel_offset_x} 0 ${caster_wheel_offset_z}" />
     </joint>
     <link name="caster_wheel">
         <visual>
             <geometry>
-                <sphere radius="0.05" />
+                <sphere radius="${caster_wheel_radius}" />
             </geometry>
-            <material name="black" />
+            <material name="white" />
         </visual>
         <collision>
             <geometry>
-                <sphere radius="0.05" />
+                <sphere radius="${caster_wheel_radius}" />
             </geometry>
         </collision>
-        <xacro:inertial_sphere mass="0.1" radius="0.05">
+        <xacro:inertial_sphere mass="${caster_wheel_mass}" radius="${caster_wheel_radius}">
             <origin xyz="0 0 0" rpy="0 0 0" />
         </xacro:inertial_sphere>
